File: uconsole-expansion-card-template-kicad-dev/uconsole-expansion-card-template/uconsole-expansion-card-template.kicad_pcb (KiCad board)
At the start: 2 copper layers, 35.8 x 77 mm, 10 parts, among them J1 EXPOSURE GPIO, J2 Camera, U1 Speaker, U2 Speaker, U3 UC EXPANSION

Commit message: Add files via upload
Parts:
- moved R1 5.73 mm to (99.3, 105.2)
- moved R2 5.73 mm to (99.3, 102.1)
- moved J2 2.35 mm to (99.6, 123.4), turned to 90 degrees
Routing:
- net GND: track 201.3 -> 129.8 mm, vias 3 -> 8
- net /CAM1_DN0: track 16.9 -> 44.0 mm
- net /CAM1_DP0: track 17.9 -> 41.6 mm
- net /CAM1_DN1: track 19.7 -> 40.4 mm
- net /SPEAKER_RN: track 67.1 -> 85.2 mm
- net /GPIO43/CAM_LED: track 69.0 -> 51.7 mm, vias 0 -> 2
- net /GPIO42/CAM_EN: track 60.6 -> 46.4 mm, vias 0 -> 2
- net /CAM1_DP1: track 20.7 -> 33.1 mm
- net /GPIO44/I2C_SDA: track 54.7 -> 44.2 mm, vias 0 -> 2
- net /CAM1_CP: track 40.8 -> 30.8 mm, vias 4 -> 0
- net /SPEAKER_RP: track 78.7 -> 69.1 mm
- net /CAM1_CN: track 26.6 -> 34.5 mm, vias 4 -> 0
- net /GPIO45/I2C_SCL: track 59.3 -> 52.1 mm
- net /CAM1_DN3: track 28.6 -> 33.5 mm, vias 0 -> 2
- net /CAM1_DN2: track 26.2 -> 30.8 mm, vias 0 -> 2
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
Commit message: Add files via upload
Parts:
- moved J2 5.69 mm to (97.3, 128.6), turned to 0 degrees
Routing:
- net /SPEAKER_RN: track 85.2 -> 61.7 mm
- net /GPIO44/I2C_SDA: track 44.2 -> 61.4 mm, vias 2 -> 0
- net /SPEAKER_RP: track 69.1 -> 84.4 mm
- net +3V3: track 57.4 -> 72.6 mm
- net /CAM1_DN0: track 44.0 -> 33.1 mm
- net +5V: track 51.4 -> 41.3 mm, vias 1 -> 2
- net /GPIO42/CAM_EN: track 46.4 -> 56.4 mm, vias 2 -> 1
- net /GPIO45/I2C_SCL: track 52.1 -> 60.2 mm, vias 1 -> 0
- net /GPIO43/CAM_LED: track 51.7 -> 59.2 mm, vias 2 -> 1
- net /CAM1_DN1: track 40.4 -> 33.2 mm
- net /SPEAKER_LN: track 42.3 -> 48.6 mm
- net /CAM1_DP0: track 41.6 -> 35.5 mm
- net /SPEAKER_LP: track 44.3 -> 40.0 mm
- net /CAM1_DN2: track 30.8 -> 33.7 mm, vias 2 -> 0
- net /CAM1_CP: track 30.8 -> 33.3 mm
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